File: pcb/led_driver.sch (KiCad schematic (older format))
At the start: 38 parts, among them P1 POWER, P2 ICSP, Q1 DMP2305U, Q2 DMP2305U, SW1 UP, SW2 DOWN, U1 PIC16(L)F616-I/ST

Commit message: Fixed missing footprint error
Parts:
- U1: footprint (none) -> Housings_SSOP:TSSOP-14_4.4x5mm_Pitch0.65mm
Changed lines of the file:
@@
 F 0 "U1" H 6200 2700 50  0000 L CNN
 F 1 "PIC16(L)F616-I/ST" H 6200 2600 50  0000 L CNN
-F 2 "" H 8000 2100 50  0000 C CNN
+F 2 "Housings_SSOP:TSSOP-14_4.4x5mm_Pitch0.65mm" H 8000 2100 50  0001 C CNN
 F 3 "" H 8000 2100 50  0000 C CNN
 	1    8000 2100

Commit message: Cleanup before sending to seedstudio
Other:
- note removed: "designed for LiIon battery\nmax 5V, min 3V (below 3V powered off by MCU)"
- note removed: "diode to avoid reset during switching the led on (voltage may drop for a while)"
Changed lines of the file:
@@
 encoding utf-8
 Sheet 1 1
-Title "Headlamp led driver"
-Date ""
-Rev "1.1"
+Title "Darkstar - Double Cree XP-G2 Headlamp "
+Date "2015-12-04"
+Rev "1.2"
 Comp "Kajus"
 Comment1 "Based on http://ww1.microchip.com/downloads/en/AppNotes/00874C.pdf"
 Comment2 "Operates at ~130kHz, designed for ~1A per led"
-Comment3 "Turns off at 3V, max input voltage is 5,3V, designed for LiIon batteries"
-Comment4 ""
+Comment3 "Turns off at 3V, max input voltage is 5,3V"
+Comment4 "LiIon batteries recommended"
 $EndDescr
 $Comp
@@
 $EndComp
 Connection ~ 8000 950
-Text Notes 7400 600  0    60   ~ 0
-diode to avoid reset during switching the led on (voltage may drop for a while)
 $Comp
 L PWR_FLAG #FLG018
@@
 	4950 2350 4950 2200
 Connection ~ 4550 2350
-Text Notes 600  1500 0    60   ~ 0
-designed for LiIon battery\nmax 5V, min 3V (below 3V powered off by MCU)
 Wire Wire Line
 	1500 700  1500 650

Commit message: Divider modified for higher stability and overcurrent protection on fw error
Parts:
- C2, C4: value 820n -> 1u
- R3, R6: value 100k -> 190k
- R4, R7: value 4k7 -> 5k6
Changed lines of the file:
@@
 P 3300 7200
 F 0 "C4" H 3310 7270 50  0000 L CNN
-F 1 "820n" H 3310 7120 50  0000 L CNN
+F 1 "1u" H 3310 7120 50  0000 L CNN
 F 2 "Capacitors_SMD:C_0805" H 3300 7200 60  0001 C CNN
 F 3 "" H 3300 7200 60  0000 C CNN
@@
 P 3050 6450
 F 0 "R6" V 3130 6450 50  0000 C CNN
-F 1 "100k" V 3050 6450 50  0000 C CNN
+F 1 "190k" V 3050 6450 50  0000 C CNN
 F 2 "Resistors_SMD:R_0805" H 3050 6450 60  0001 C CNN
 F 3 "" H 3050 6450 60  0000 C CNN
@@
 P 1450 6450
 F 0 "R3" V 1530 6450 50  0000 C CNN
-F 1 "100k" V 1450 6450 50  0000 C CNN
+F 1 "190k" V 1450 6450 50  0000 C CNN
 F 2 "Resistors_SMD:R_0805" H 1450 6450 60  0001 C CNN
 F 3 "" H 1450 6450 60  0000 C CNN
@@
 P 1700 7150
 F 0 "C2" H 1710 7220 50  0000 L CNN
-F 1 "820n" H 1710 7070 50  0000 L CNN
+F 1 "1u" H 1710 7070 50  0000 L CNN
 F 2 "Capacitors_SMD:C_0805" H 1700 7150 60  0001 C CNN
 F 3 "" H 1700 7150 60  0000 C CNN
@@
 P 3050 7200
 F 0 "R7" V 3130 7200 50  0000 C CNN
-F 1 "4k7" V 3050 7200 50  0000 C CNN
+F 1 "5k6" V 3050 7200 50  0000 C CNN
 F 2 "Resistors_SMD:R_0805" H 3050 7200 60  0001 C CNN
 F 3 "" H 3050 7200 60  0000 C CNN
@@
 P 1450 7150
 F 0 "R4" V 1530 7150 50  0000 C CNN
-F 1 "4k7" V 1450 7150 50  0000 C CNN
+F 1 "5k6" V 1450 7150 50  0000 C CNN
 F 2 "Resistors_SMD:R_0805" H 1450 7150 60  0001 C CNN
 F 3 "" H 1450 7150 60  0000 C CNN

Commit message: Fixed resistor not in E12
Parts:
- R3, R6: value 190k -> 180k
Changed lines of the file:
@@
 P 3050 6450
 F 0 "R6" V 3130 6450 50  0000 C CNN
-F 1 "190k" V 3050 6450 50  0000 C CNN
+F 1 "180k" V 3050 6450 50  0000 C CNN
 F 2 "Resistors_SMD:R_0805" H 3050 6450 60  0001 C CNN
 F 3 "" H 3050 6450 60  0000 C CNN
@@
 P 1450 6450
 F 0 "R3" V 1530 6450 50  0000 C CNN
-F 1 "190k" V 1450 6450 50  0000 C CNN
+F 1 "180k" V 1450 6450 50  0000 C CNN
 F 2 "Resistors_SMD:R_0805" H 1450 6450 60  0001 C CNN
 F 3 "" H 1450 6450 60  0000 C CNN
